File: Vernier_Vamp-200mA/DAC.sch (KiCad schematic (older format))
At the start: 56 parts, among them U10 OPA2277, U11 OPA2277, U7 LTC6655-2.5, U8 DAC8814, U9 OPA2277

Commit message: Coil driver version 1.0B
Updated coil driver 200mA version with fixes requested by Iain.
Connections:
- net labels added: +7.5V, -7.5V
- net labels removed: +8V, -8V
Other:
- note added: "DAC decoupling\n"
- note added: "OP-AMP decoupling"
- moved on the sheet: C14, C15, C16, C17, C18, C19, C20, C21, C22, C23, C24, C25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
