File: Vernier_Vamp-200mA/Vernier_Vamp-200mA.kicad_pcb (KiCad board)
At the start: 4 copper layers, 160 x 99.5 mm, 236 parts, among them J1 Conn_01x02, J2 RJ45, J3 Screw_Terminal_01x04, J4 Conn_02x07_Odd_Even, J5 Channel 3, J6 Channel 2, J7 Channel 1, J8 RF_Shield_Two_Pieces, J9 Conn_01x02, Q1 Si4447ADY, Q2 IRF8707PbF, Q3 2SC5566, Q4 2SA2013, Q5 2SC5566, Q6 2SA2013, Q7 2SC5566, Q8 2SA2013, SW1 DPDT_Hirose, U1 LM4040DBZ-5, U10 OPA2277, U11 OPA2277, U12 OPA2277, U13 OPA2277, U14 OPA2277, U2 LM4040DBZ-5, U3 LM393, U4 TPS7A470x, U5 TPS7A470x, U6 TPS7A33, U7 LTC6655-2.5, U8 DAC8814, U9 OPA2277

Commit message: Addition of test points onto the bias circuitry
-Addition of test points onto the bias circuitry (HCCD)
-Silkscreen update (LCCD)
Parts:
- added TP55: TestPoint_Probe, TestPoint:TestPoint_Pad_D1.0mm, F.Cu at (144.3, 71.0)
- added TP56: TestPoint_Probe, TestPoint:TestPoint_Pad_D1.0mm, F.Cu at (144.3, 65.8)
- added TP57: TestPoint_Probe, TestPoint:TestPoint_Pad_D1.0mm, F.Cu at (144.3, 58.1)
- added TP58: TestPoint_Probe, TestPoint:TestPoint_Pad_D1.0mm, F.Cu at (144.3, 52.9)
- added TP59: TestPoint_Probe, TestPoint:TestPoint_Pad_D1.0mm, F.Cu at (144.3, 96.8)
- added TP60: TestPoint_Probe, TestPoint:TestPoint_Pad_D1.0mm, F.Cu at (144.3, 91.5)
- added TP61: TestPoint_Probe, TestPoint:TestPoint_Pad_D1.0mm, F.Cu at (144.3, 83.9)
- added TP62: TestPoint_Probe, TestPoint:TestPoint_Pad_D1.0mm, F.Cu at (144.3, 78.6)
- added TP63: TestPoint_Probe, TestPoint:TestPoint_Pad_D1.0mm, F.Cu at (144.3, 122.8)
- added TP64: TestPoint_Probe, TestPoint:TestPoint_Pad_D1.0mm, F.Cu at (144.3, 117.5)
- added TP65: TestPoint_Probe, TestPoint:TestPoint_Pad_D1.0mm, F.Cu at (142.2, 113.5)
- added TP66: TestPoint_Probe, TestPoint:TestPoint_Pad_D1.0mm, F.Cu at (144.3, 104.0)
Connections:
- A1 pad 1: (no net) -> Net-(A1-Pad1)
- A1 pad 17: (no net) -> Net-(A1-Pad17)
- A1 pad 18: (no net) -> Net-(A1-Pad18)
- A1 pad 2: (no net) -> Net-(A1-Pad2)
- A1 pad 20: (no net) -> Net-(A1-Pad20)
- A1 pad 21: (no net) -> Net-(A1-Pad21)
- A1 pad 22: (no net) -> Net-(A1-Pad22)
- A1 pad 23: (no net) -> Net-(A1-Pad23)
- A1 pad 24: (no net) -> Net-(A1-Pad24)
- A1 pad 25: (no net) -> Net-(A1-Pad25)
- A1 pad 26: (no net) -> Net-(A1-Pad26)
- A1 pad 28: (no net) -> Net-(A1-Pad28)
- A1 pad 3: (no net) -> Net-(A1-Pad3)
- A1 pad 5: (no net) -> Net-(A1-Pad5)
- A1 pad 6: (no net) -> Net-(A1-Pad6)
- A1 pad 7: (no net) -> Net-(A1-Pad7)
- A1 pad 8: (no net) -> Net-(A1-Pad8)
- A1 pad 9: (no net) -> Net-(A1-Pad9)
- RV1 pad 3: (no net) -> Net-(RV1-Pad3)
- RV2 pad 1: (no net) -> Net-(RV2-Pad1)
- RV3 pad 3: (no net) -> Net-(RV3-Pad3)
- RV4 pad 1: (no net) -> Net-(RV4-Pad1)
- RV5 pad 3: (no net) -> Net-(RV5-Pad3)
- RV6 pad 1: (no net) -> Net-(RV6-Pad1)
- U4 pad 11: (no net) -> Net-(U4-Pad11)
- U4 pad 4: (no net) -> Net-(U4-Pad4)
- U4 pad 5: (no net) -> Net-(U4-Pad5)
- U5 pad 11: (no net) -> Net-(U5-Pad11)
- U5 pad 12: (no net) -> Net-(U5-Pad12)
- U5 pad 4: (no net) -> Net-(U5-Pad4)
- U5 pad 5: (no net) -> Net-(U5-Pad5)
- U5 pad 8: (no net) -> Net-(U5-Pad8)
- U5 pad 9: (no net) -> Net-(U5-Pad9)
Routing:
- net Net-(D9-Pad2): track 7.03 -> 13.0 mm
- net -7V5: track 59.7 -> 63.7 mm, vias 55 -> 58
- net +7V5: track 75.7 -> 79.6 mm, vias 59 -> 62
- net Net-(D8-Pad1): track 11.0 -> 13.0 mm
- net Net-(D9-Pad1): track 11.0 -> 12.9 mm
- net Net-(D8-Pad2): track 7.03 -> 8.93 mm
- net Net-(D7-Pad1): track 11.0 -> 12.8 mm
- net Net-(D7-Pad2): track 7.03 -> 8.84 mm
