File: High_Current_Driver/High_Current_Driver.kicad_pcb (KiCad board)
At the start: 4 copper layers, 160 x 99.5 mm, 248 parts, among them J1 Conn_01x02, J2 RJ45, J3 Screw_Terminal_01x04, J4 Conn_02x07_Odd_Even, J5 Channel 3, J6 Channel 2, J7 Channel 1, J8 RF_Shield_Two_Pieces, J9 Conn_01x02, Q1 Si4447ADY, Q2 IRF8707PbF, Q3 2SC5566, Q4 2SA2013, Q5 2SC5566, Q6 2SA2013, Q7 2SC5566, Q8 2SA2013, SW1 DPDT_Hirose, U1 LM4040DBZ-5, U10 OPA2277, U11 OPA2277, U12 OPA2277, U13 OPA2277, U14 OPA2277, U2 LM4040DBZ-5, U3 LM393, U4 TPS7A470x, U5 TPS7A470x, U6 TPS7A33, U7 LTC6655-2.5, U8 DAC8814, U9 OPA2277

Commit message: HCD amplifier update
- Updated OPA2277 amplifiers to OPA2210 that were actually populated on the boards.
Parts:
- U10, U11, U12, U13, U14, U9: value OPA2277 -> OPA2210
Connections:
- A1 pad 1: Net-(A1-Pad1) -> (no net)
- A1 pad 17: Net-(A1-Pad17) -> (no net)
- A1 pad 18: Net-(A1-Pad18) -> (no net)
- A1 pad 2: Net-(A1-Pad2) -> (no net)
- A1 pad 20: Net-(A1-Pad20) -> (no net)
- A1 pad 21: Net-(A1-Pad21) -> (no net)
- A1 pad 22: Net-(A1-Pad22) -> (no net)
- A1 pad 23: Net-(A1-Pad23) -> (no net)
- A1 pad 24: Net-(A1-Pad24) -> (no net)
- A1 pad 25: Net-(A1-Pad25) -> (no net)
- A1 pad 26: Net-(A1-Pad26) -> (no net)
- A1 pad 28: Net-(A1-Pad28) -> (no net)
- A1 pad 3: Net-(A1-Pad3) -> (no net)
- A1 pad 5: Net-(A1-Pad5) -> (no net)
- A1 pad 6: Net-(A1-Pad6) -> (no net)
- A1 pad 7: Net-(A1-Pad7) -> (no net)
- A1 pad 8: Net-(A1-Pad8) -> (no net)
- A1 pad 9: Net-(A1-Pad9) -> (no net)
- RV1 pad 3: Net-(RV1-Pad3) -> (no net)
- RV2 pad 1: Net-(RV2-Pad1) -> (no net)
- RV3 pad 3: Net-(RV3-Pad3) -> (no net)
- RV4 pad 1: Net-(RV4-Pad1) -> (no net)
- RV5 pad 3: Net-(RV5-Pad3) -> (no net)
- RV6 pad 1: Net-(RV6-Pad1) -> (no net)
- U4 pad 11: Net-(U4-Pad11) -> (no net)
- U4 pad 4: Net-(U4-Pad4) -> (no net)
- U4 pad 5: Net-(U4-Pad5) -> (no net)
- U5 pad 11: Net-(U5-Pad11) -> (no net)
- U5 pad 12: Net-(U5-Pad12) -> (no net)
- U5 pad 4: Net-(U5-Pad4) -> (no net)
- U5 pad 5: Net-(U5-Pad5) -> (no net)
- U5 pad 8: Net-(U5-Pad8) -> (no net)
- U5 pad 9: Net-(U5-Pad9) -> (no net)
