File: Hardware/PCBs/High_Current_Driver/Battery_Management.sch (KiCad schematic (older format))
At the start: 49 parts, among them J4 Conn_02x07_Odd_Even, Q1 Si4447ADY, Q2 IRF8707PbF, SW1 DPDT_Hirose, U1 LM4040DBZ-5, U2 LM4040DBZ-5, U3 LM393

Commit message: Switch to common shared library
Parts:
- D1, D2, D3, D4: symbol SMBJ15A:SMBJ15A -> vernier_current_driver:SMBJ15A
- Q1: symbol Si4447ADY:Si4447ADY -> vernier_current_driver:Si4447ADY
- Q2: symbol IRF8707PbF:IRF8707PbF -> vernier_current_driver:IRF8707PbF
- SW1: symbol SW_DPDT_Hirose:DPDT_Hirose -> vernier_current_driver:DPDT_Hirose
Changed lines of the file:
@@
 $EndComp
 $Comp
-L SMBJ15A:SMBJ15A D?
+L vernier_current_driver:SMBJ15A D?
 U 1 1 5EB425D6
 P 4200 1600
@@
 $EndComp
 $Comp
-L IRF8707PbF:IRF8707PbF Q?
+L vernier_current_driver:IRF8707PbF Q?
 U 1 1 5EB425F5
 P 2950 2950
@@
 $EndComp
 $Comp
-L Si4447ADY:Si4447ADY Q?
+L vernier_current_driver:Si4447ADY Q?
 U 1 1 5EB425FB
 P 2950 1200
@@
 	4200 3700 4200 3450
 $Comp
-L SMBJ15A:SMBJ15A D?
+L vernier_current_driver:SMBJ15A D?
 U 1 1 5EB4260A
 P 4200 3300
@@
 	1850 2900 2750 2900
 $Comp
-L SMBJ15A:SMBJ15A D?
+L vernier_current_driver:SMBJ15A D?
 U 1 1 5EB4261D
 P 3400 1400
@@
 $EndComp
 $Comp
-L SMBJ15A:SMBJ15A D?
+L vernier_current_driver:SMBJ15A D?
 U 1 1 5EB4263E
 P 3400 3100
@@
 Connection ~ 7350 1850
 $Comp
-L SW_DPDT_Hirose:DPDT_Hirose SW?
+L vernier_current_driver:DPDT_Hirose SW?
 U 2 1 5EB42722
 P 7050 1000
@@
 +12VDC_bat
 $Comp
-L custom_power_rails:+12V_batt_post #PWR0176
+L vernier_current_driver:+12V_batt_post #PWR0176
 U 1 1 5ECA0162
 P 7350 1000
@@
 $EndComp
 $Comp
-L custom_power_rails:+7.5V #PWR?
+L vernier_current_driver:+7.5V #PWR?
 U 1 1 5EFE147B
 P 8500 1000
@@
 $EndComp
 $Comp
-L custom_power_rails:-7.5V #PWR?
+L vernier_current_driver:-7.5V #PWR?
 U 1 1 5EFFB5B2
 P 10150 1000
@@
 $EndComp
 $Comp
-L SW_DPDT_Hirose:DPDT_Hirose SW?
+L vernier_current_driver:DPDT_Hirose SW?
 U 1 1 5EB4271C
 P 7050 1650
