File: Hardware/PCBs/High_Current_Driver/Channel_Outputs.sch (KiCad schematic (older format))
At the start: 99 parts, among them Q3 2SC5566, Q4 2SA2013, Q5 2SC5566, Q6 2SA2013, Q7 2SC5566, Q8 2SA2013, U12 OPA2210, U13 OPA2210, U14 OPA2210

Commit message: Switch to common footprint library
Parts:
- R48, R49, R55: footprint WSM2-13R0-FTR-LF:WSM2 13R0 FTR-LF -> vernier_current_driver:WSM2_13R0_FTR-LF
Changed lines of the file:
@@
 F 0 "R49" H 5209 5146 50  0000 L CNN
 F 1 "13R" H 5209 5055 50  0000 L CNN
-F 2 "WSM2-13R0-FTR-LF:WSM2 13R0 FTR-LF" H 5150 5100 50  0001 C CNN
+F 2 "vernier_current_driver:WSM2_13R0_FTR-LF" H 5150 5100 50  0001 C CNN
 F 3 "~" H 5150 5100 50  0001 C CNN
 	1    5150 5100
@@
 F 0 "R48" H 5209 2696 50  0000 L CNN
 F 1 "13R" H 5209 2605 50  0000 L CNN
-F 2 "WSM2-13R0-FTR-LF:WSM2 13R0 FTR-LF" H 5150 2650 50  0001 C CNN
+F 2 "vernier_current_driver:WSM2_13R0_FTR-LF" H 5150 2650 50  0001 C CNN
 F 3 "~" H 5150 2650 50  0001 C CNN
 	1    5150 2650
@@
 F 0 "R55" H 10509 2696 50  0000 L CNN
 F 1 "13R" H 10509 2605 50  0000 L CNN
-F 2 "WSM2-13R0-FTR-LF:WSM2 13R0 FTR-LF" H 10450 2650 50  0001 C CNN
+F 2 "vernier_current_driver:WSM2_13R0_FTR-LF" H 10450 2650 50  0001 C CNN
 F 3 "~" H 10450 2650 50  0001 C CNN
 	1    10450 2650

Commit message: Switch to common shared library
Parts:
- Q3, Q5, Q7: symbol 2SA2013_2SC5566:2SC5566 -> vernier_current_driver:2SC5566
- Q4, Q6, Q8: symbol 2SA2013_2SC5566:2SA2013 -> vernier_current_driver:2SA2013
- U12, U13, U14: symbol OPA2210:OPA2210 -> vernier_current_driver:OPA2210
Changed lines of the file:
@@
 $EndDescr
 $Comp
-L OPA2210:OPA2210 U12
+L vernier_current_driver:OPA2210 U12
 U 1 1 5EA48838
 P 2450 2100
@@
 $EndComp
 $Comp
-L OPA2210:OPA2210 U12
+L vernier_current_driver:OPA2210 U12
 U 3 1 5EA4AA3C
 P 2450 2100
@@
 4Q_DAC_OUT_1
 $Comp
-L OPA2210:OPA2210 U13
+L vernier_current_driver:OPA2210 U13
 U 1 1 5EA9B480
 P 2450 4550
@@
 $EndComp
 $Comp
-L OPA2210:OPA2210 U13
+L vernier_current_driver:OPA2210 U13
 U 3 1 5EA9B486
 P 2450 4550
@@
 4Q_DAC_OUT_2
 $Comp
-L OPA2210:OPA2210 U14
+L vernier_current_driver:OPA2210 U14
 U 1 1 5EAB3D14
 P 7750 2100
@@
 $EndComp
 $Comp
-L OPA2210:OPA2210 U14
+L vernier_current_driver:OPA2210 U14
 U 3 1 5EAB3D1A
 P 7750 2100
@@
 	5150 4750 5300 4750
 $Comp
-L OPA2210:OPA2210 U13
+L vernier_current_driver:OPA2210 U13
 U 2 1 60341939
 P 3350 4050
@@
 $EndComp
 $Comp
-L OPA2210:OPA2210 U14
+L vernier_current_driver:OPA2210 U14
 U 2 1 6034B68E
 P 8650 1600
@@
 $EndComp
 $Comp
-L custom_power_rails:+7.5V #PWR?
+L vernier_current_driver:+7.5V #PWR?
 U 1 1 5EEC72C9
 P 2350 1800
@@
 $EndComp
 $Comp
-L custom_power_rails:+7.5V #PWR?
+L vernier_current_driver:+7.5V #PWR?
 U 1 1 5EEF4C71
 P 2350 4250
@@
 $EndComp
 $Comp
-L custom_power_rails:+7.5V #PWR?
+L vernier_current_driver:+7.5V #PWR?
 U 1 1 5EF1348E
 P 7650 1800
@@
 $EndComp
 $Comp
-L custom_power_rails:-7.5V #PWR?
+L vernier_current_driver:-7.5V #PWR?
 U 1 1 5EF22BC2
 P 2350 4850
@@
 $EndComp
 $Comp
-L custom_power_rails:-7.5V #PWR?
+L vernier_current_driver:-7.5V #PWR?
 U 1 1 5EF413DB
 P 7650 2400
@@
 $EndComp
 $Comp
-L custom_power_rails:-7.5V #PWR?
+L vernier_current_driver:-7.5V #PWR?
 U 1 1 5EF5F0FD
 P 2350 2400
@@
 $EndComp
 $Comp
-L custom_power_rails:-7.5V #PWR?
+L vernier_current_driver:-7.5V #PWR?
 U 1 1 5EFAA3CB
 P 850 7500
@@
 $EndComp
 $Comp
-L custom_power_rails:+7.5V #PWR?
+L vernier_current_driver:+7.5V #PWR?
 U 1 1 5EFC850A
 P 900 6200
@@
 OP-AMP decoupling
 $Comp
-L 2SA2013_2SC5566:2SA2013 Q6
+L vernier_current_driver:2SA2013 Q6
 U 1 1 60ACAE0A
 P 4750 4450
@@
 $EndComp
 $Comp
-L 2SA2013_2SC5566:2SC5566 Q5
+L vernier_current_driver:2SC5566 Q5
 U 1 1 60ACD0CB
 P 4750 3650
@@
 	5150 4100 5050 4100
 $Comp
-L custom_power_rails:+7.5V #PWR?
+L vernier_current_driver:+7.5V #PWR?
 U 1 1 60E486A8
 P 4750 3150
@@
 $EndComp
 $Comp
-L custom_power_rails:+7.5V #PWR?
+L vernier_current_driver:+7.5V #PWR?
 U 1 1 60E7132F
 P 4100 3150
@@
 	4100 3150 4100 3200
 $Comp
-L custom_power_rails:-7.5V #PWR?
+L vernier_current_driver:-7.5V #PWR?
 U 1 1 60E9B9E1
 P 4100 4950
@@
 $EndComp
 $Comp
-L custom_power_rails:-7.5V #PWR?
+L vernier_current_driver:-7.5V #PWR?
 U 1 1 60EA960C
 P 4750 4950
@@
 	5150 2300 5300 2300
 $Comp
-L 2SA2013_2SC5566:2SA2013 Q4
+L vernier_current_driver:2SA2013 Q4
 U 1 1 6139A770
 P 4750 2000
@@
 $EndComp
 $Comp
-L 2SA2013_2SC5566:2SC5566 Q3
+L vernier_current_driver:2SC5566 Q3
 U 1 1 6139A776
 P 4750 1200
@@
 	5150 1650 5050 1650
 $Comp
-L custom_power_rails:+7.5V #PWR?
+L vernier_current_driver:+7.5V #PWR?
 U 1 1 6139A7CD
 P 4750 700
@@
 $EndComp
 $Comp
-L custom_power_rails:+7.5V #PWR?
+L vernier_current_driver:+7.5V #PWR?
 U 1 1 6139A7D3
 P 4100 700
@@
 	4100 700  4100 750
 $Comp
-L custom_power_rails:-7.5V #PWR?
+L vernier_current_driver:-7.5V #PWR?
 U 1 1 6139A7DB
 P 4100 2500
@@
 $EndComp
 $Comp
-L custom_power_rails:-7.5V #PWR?
+L vernier_current_driver:-7.5V #PWR?
 U 1 1 6139A7E1
 P 4750 2500
@@
 	3700 1600 3650 1600
 $Comp
-L OPA2210:OPA2210 U12
+L vernier_current_driver:OPA2210 U12
 U 2 1 60337A87
 P 3350 1600
@@
 	10450 2300 10600 2300
 $Comp
-L 2SA2013_2SC5566:2SA2013 Q8
+L vernier_current_driver:2SA2013 Q8
 U 1 1 615FDB22
 P 10050 2000
@@
 $EndComp
 $Comp
-L 2SA2013_2SC5566:2SC5566 Q7
+L vernier_current_driver:2SC5566 Q7
 U 1 1 615FDB28
 P 10050 1200
@@
 	10450 1650 10350 1650
 $Comp
-L custom_power_rails:+7.5V #PWR?
+L vernier_current_driver:+7.5V #PWR?
 U 1 1 615FDB7F
 P 10050 700
@@
 $EndComp
 $Comp
-L custom_power_rails:+7.5V #PWR?
+L vernier_current_driver:+7.5V #PWR?
 U 1 1 615FDB85
 P 9400 700
@@
 	9400 700  9400 750
 $Comp
-L custom_power_rails:-7.5V #PWR?
+L vernier_current_driver:-7.5V #PWR?
 U 1 1 615FDB8D
 P 9400 2500
@@
 $EndComp
 $Comp
-L custom_power_rails:-7.5V #PWR?
+L vernier_current_driver:-7.5V #PWR?
 U 1 1 615FDB93
 P 10050 2500
