File: Hardware/PCBs/High_Current_Driver/High_Current_Driver.sch (KiCad schematic (older format))
At the start: 7 parts, among them J1 Conn_01x02, J2 RJ45, J3 Screw_Terminal_01x04, J5 Channel 3, J6 Channel 2, J7 Channel 1, J8 RF_Shield_Two_Pieces

Commit message: Switch to common footprint library
Parts:
- J1: footprint Dummy_conn_01x02:PinSocket_1x02_P1.00mm_Vertical_CUSTOM_CYD -> vernier_current_driver:PinSocket_1x02_P1.00mm_Vertical_CUSTOM_CYD
- J8: footprint MS570-10F:MS570-10S -> vernier_current_driver:MS570-10S
Changed lines of the file:
@@
 F 0 "J1" H 8780 4192 50  0000 L CNN
 F 1 "Conn_01x02" H 8780 4101 50  0000 L CNN
-F 2 "Dummy_conn_01x02:PinSocket_1x02_P1.00mm_Vertical_CUSTOM_CYD" H 8700 4200 50  0001 C CNN
+F 2 "vernier_current_driver:PinSocket_1x02_P1.00mm_Vertical_CUSTOM_CYD" H 8700 4200 50  0001 C CNN
 F 3 "~" H 8700 4200 50  0001 C CNN
 	1    8700 4200
@@
 F 0 "J8" H 2030 6014 50  0000 L CNN
 F 1 "RF_Shield_Two_Pieces" H 2030 5923 50  0000 L CNN
-F 2 "MS570-10F:MS570-10S" H 1300 5850 50  0001 C CNN
+F 2 "vernier_current_driver:MS570-10S" H 1300 5850 50  0001 C CNN
 F 3 "~" H 1300 5850 50  0001 C CNN
 	1    1300 5950
