File: Hardware/PCBs/High_Current_Driver/MCU.sch (KiCad schematic (older format))
At the start: 13 parts, among them J9 Conn_01x02

Commit message: Switch to common shared library
Changed lines of the file:
@@
 	4600 2550 4600 2650
 $Comp
-L custom_power_rails:+12V_batt_post #PWR?
+L vernier_current_driver:+12V_batt_post #PWR?
 U 1 1 5ECA4E39
 P 4600 2550
