File: Hardware/PCBs/High_Current_Driver/Power.sch (KiCad schematic (older format))
At the start: 19 parts, among them U4 TPS7A470x, U5 TPS7A470x, U6 TPS7A33

Commit message: Switch to common shared library
Parts:
- U4, U5: symbol TPS74A4700:TPS7A4700 -> vernier_current_driver:TPS7A4700
- U6: symbol TPS7A33:TPS7A33 -> vernier_current_driver:TPS7A33
Changed lines of the file:
@@
 	6550 5350 6950 5350
 $Comp
-L TPS7A33:TPS7A33 U6
+L vernier_current_driver:TPS7A33 U6
 U 1 1 5E321ECA
 P 5650 5250
@@
 	5150 5350 4250 5350
 $Comp
-L TPS74A4700:TPS7A4700 U5
+L vernier_current_driver:TPS7A4700 U5
 U 1 1 5E4EDE9C
 P 5650 3050
@@
 $EndComp
 $Comp
-L TPS74A4700:TPS7A4700 U4
+L vernier_current_driver:TPS7A4700 U4
 U 1 1 5E30DC9B
 P 5650 950
@@
 	2700 1050 2850 1050
 $Comp
-L custom_power_rails:-7.5V #PWR0113
+L vernier_current_driver:-7.5V #PWR0113
 U 1 1 5ECDFF18
 P 7300 5650
@@
 	7350 500  7350 2450
 $Comp
-L custom_power_rails:+7.5V #PWR0120
+L vernier_current_driver:+7.5V #PWR0120
 U 1 1 5ECE6050
 P 7200 800
