File: Hardware/PCBs/Low_Current_Driver/Battery_Management.sch (KiCad schematic (older format))
At the start: 49 parts, among them J4 Conn_02x07_Odd_Even, Q1 Si4447ADY, Q2 IRF8707PbF, SW1 DPDT_Hirose, U1 LM4040DBZ-5, U2 LM4040DBZ-5, U3 LM393

Commit message: Switch to common shared library
Parts:
- D3, D4, D5, D6: symbol SMBJ15A:SMBJ15A -> vernier_current_driver:SMBJ15A
- Q1: symbol Si4447ADY:Si4447ADY -> vernier_current_driver:Si4447ADY
- Q2: symbol IRF8707PbF:IRF8707PbF -> vernier_current_driver:IRF8707PbF
- SW1: symbol SW_DPDT_Hirose:DPDT_Hirose -> vernier_current_driver:DPDT_Hirose
Changed lines of the file:
@@
 $EndComp
 $Comp
-L SMBJ15A:SMBJ15A D?
+L vernier_current_driver:SMBJ15A D?
 U 1 1 5EC3DDB6
 P 4100 1600
@@
 $EndComp
 $Comp
-L IRF8707PbF:IRF8707PbF Q?
+L vernier_current_driver:IRF8707PbF Q?
 U 1 1 5EC3DDD5
 P 2850 2950
@@
 $EndComp
 $Comp
-L Si4447ADY:Si4447ADY Q?
+L vernier_current_driver:Si4447ADY Q?
 U 1 1 5EC3DDDB
 P 2850 1200
@@
 	4100 3700 4100 3450
 $Comp
-L SMBJ15A:SMBJ15A D?
+L vernier_current_driver:SMBJ15A D?
 U 1 1 5EC3DDEA
 P 4100 3300
@@
 	1750 2900 2650 2900
 $Comp
-L SMBJ15A:SMBJ15A D?
+L vernier_current_driver:SMBJ15A D?
 U 1 1 5EC3DDFD
 P 3300 1400
@@
 $EndComp
 $Comp
-L SMBJ15A:SMBJ15A D?
+L vernier_current_driver:SMBJ15A D?
 U 1 1 5EC3DE1E
 P 3300 3100
@@
 	7650 1750 7700 1750
 $Comp
-L SW_DPDT_Hirose:DPDT_Hirose SW?
+L vernier_current_driver:DPDT_Hirose SW?
 U 1 1 5EC516F5
 P 7350 1550
@@
 $EndComp
 $Comp
-L SW_DPDT_Hirose:DPDT_Hirose SW?
+L vernier_current_driver:DPDT_Hirose SW?
 U 2 1 5EC516FB
 P 7350 900
@@
 	5250 4850 5950 4850
 $Comp
-L custom_power_rails:-7.5V #PWR0140
+L vernier_current_driver:-7.5V #PWR0140
 U 1 1 5ECB7631
 P 10300 850
@@
 $EndComp
 $Comp
-L custom_power_rails:+7.5V #PWR0141
+L vernier_current_driver:+7.5V #PWR0141
 U 1 1 5ECB832C
 P 8700 950
@@
 $EndComp
 $Comp
-L custom_power_rails:+12V_batt_post #PWR0142
+L vernier_current_driver:+12V_batt_post #PWR0142
 U 1 1 5ECBF1C0
 P 7650 900
