File: Hardware/PCBs/Low_Current_Driver/Channel_Outputs.sch (KiCad schematic (older format))
At the start: 45 parts, among them U12 OPA2210, U13 OPA2210, U14 OPA2210

Commit message: Switch to common shared library
Parts:
- U12, U13, U14: symbol OPA2210:OPA2210 -> vernier_current_driver:OPA2210
Changed lines of the file:
@@
 $EndDescr
 $Comp
-L OPA2210:OPA2210 U12
+L vernier_current_driver:OPA2210 U12
 U 1 1 5EA48838
 P 4850 2100
@@
 $EndComp
 $Comp
-L OPA2210:OPA2210 U12
+L vernier_current_driver:OPA2210 U12
 U 3 1 5EA4AA3C
 P 4850 2100
@@
 4Q_DAC_OUT_1
 $Comp
-L OPA2210:OPA2210 U13
+L vernier_current_driver:OPA2210 U13
 U 1 1 5EA9B480
 P 4850 4500
@@
 $EndComp
 $Comp
-L OPA2210:OPA2210 U13
+L vernier_current_driver:OPA2210 U13
 U 3 1 5EA9B486
 P 4850 4500
@@
 4Q_DAC_OUT_2
 $Comp
-L OPA2210:OPA2210 U14
+L vernier_current_driver:OPA2210 U14
 U 1 1 5EAB3D14
 P 4850 6900
@@
 $EndComp
 $Comp
-L OPA2210:OPA2210 U14
+L vernier_current_driver:OPA2210 U14
 U 3 1 5EAB3D1A
 P 4850 6900
@@
 Connection ~ 6750 1050
 $Comp
-L custom_power_rails:+7.5V #PWR?
+L vernier_current_driver:+7.5V #PWR?
 U 1 1 5EFDFA63
 P 1050 6250
@@
 $EndComp
 $Comp
-L custom_power_rails:+7.5V #PWR?
+L vernier_current_driver:+7.5V #PWR?
 U 1 1 5EFE4517
 P 4750 6600
@@
 $EndComp
 $Comp
-L custom_power_rails:+7.5V #PWR?
+L vernier_current_driver:+7.5V #PWR?
 U 1 1 5EFE9018
 P 4750 4200
@@
 $EndComp
 $Comp
-L custom_power_rails:+7.5V #PWR?
+L vernier_current_driver:+7.5V #PWR?
 U 1 1 5EFEDB22
 P 4750 1800
@@
 $EndComp
 $Comp
-L custom_power_rails:-7.5V #PWR?
+L vernier_current_driver:-7.5V #PWR?
 U 1 1 5F0497FE
 P 1000 7550
@@
 $EndComp
 $Comp
-L custom_power_rails:-7.5V #PWR?
+L vernier_current_driver:-7.5V #PWR?
 U 1 1 5F0528F2
 P 4750 2400
@@
 $EndComp
 $Comp
-L custom_power_rails:-7.5V #PWR?
+L vernier_current_driver:-7.5V #PWR?
 U 1 1 5F0571F5
 P 4750 4800
@@
 $EndComp
 $Comp
-L custom_power_rails:-7.5V #PWR?
+L vernier_current_driver:-7.5V #PWR?
 U 1 1 5F060C92
 P 4750 7200
@@
 	6750 1050 6750 1550
 $Comp
-L OPA2210:OPA2210 U12
+L vernier_current_driver:OPA2210 U12
 U 2 1 60337A87
 P 6450 1550
@@
 Connection ~ 6750 3950
 $Comp
-L OPA2210:OPA2210 U13
+L vernier_current_driver:OPA2210 U13
 U 2 1 5FBB9E45
 P 6450 3950
@@
 Connection ~ 6750 6350
 $Comp
-L OPA2210:OPA2210 U14
+L vernier_current_driver:OPA2210 U14
 U 2 1 6034B68E
 P 6450 6350
