File: Hardware/PCBs/Low_Current_Driver/DAC.sch (KiCad schematic (older format))
At the start: 56 parts, among them U10 OPA2210, U11 OPA2210, U7 LTC6655-2.5, U8 DAC8814, U9 OPA2210

Commit message: Switch to common shared library
Parts:
- U10, U11, U9: symbol OPA2210:OPA2210 -> vernier_current_driver:OPA2210
- U7: symbol DAC8814:LTC6655-2.5 -> vernier_current_driver:LTC6655-2.5
- U8: symbol DAC8814:DAC8814 -> vernier_current_driver:DAC8814
Changed lines of the file:
@@
 	5900 4550 5450 4700
 $Comp
-L OPA2210:OPA2210 U10
+L vernier_current_driver:OPA2210 U10
 U 1 1 5EEB021E
 P 7700 3350
@@
 $EndComp
 $Comp
-L OPA2210:OPA2210 U11
+L vernier_current_driver:OPA2210 U11
 U 1 1 5EECED37
 P 7700 4750
@@
 $EndComp
 $Comp
-L OPA2210:OPA2210 U9
+L vernier_current_driver:OPA2210 U9
 U 2 1 5EECED3D
 P 9500 2050
@@
 $EndComp
 $Comp
-L OPA2210:OPA2210 U11
+L vernier_current_driver:OPA2210 U11
 U 3 1 5EECED43
 P 7700 4750
@@
 $EndComp
 $Comp
-L OPA2210:OPA2210 U11
+L vernier_current_driver:OPA2210 U11
 U 2 1 5EED36F8
 P 9500 4850
@@
 $EndComp
 $Comp
-L OPA2210:OPA2210 U9
+L vernier_current_driver:OPA2210 U9
 U 3 1 5EED36FE
 P 7700 1950
@@
 $EndComp
 $Comp
-L OPA2210:OPA2210 U9
+L vernier_current_driver:OPA2210 U9
 U 1 1 5EED36F2
 P 7700 1950
@@
 $EndComp
 $Comp
-L DAC8814:DAC8814 U8
+L vernier_current_driver:DAC8814 U8
 U 1 1 5EE568AF
 P 5650 2750
@@
 	9900 2950 9900 3450
 $Comp
-L OPA2210:OPA2210 U10
+L vernier_current_driver:OPA2210 U10
 U 2 1 5EEB1B26
 P 9500 3450
@@
 	5500 2550 5550 2550
 $Comp
-L DAC8814:LTC6655-2.5 U7
+L vernier_current_driver:LTC6655-2.5 U7
 U 1 1 5F056C56
 P 1700 1150
@@
 Connection ~ 5250 4550
 $Comp
-L custom_power_rails:+7.5V #PWR?
+L vernier_current_driver:+7.5V #PWR?
 U 1 1 5EF43E88
 P 750 1100
@@
 $EndComp
 $Comp
-L custom_power_rails:+7.5V #PWR?
+L vernier_current_driver:+7.5V #PWR?
 U 1 1 5EF6397B
 P 7600 4450
@@
 $EndComp
 $Comp
-L custom_power_rails:+7.5V #PWR?
+L vernier_current_driver:+7.5V #PWR?
 U 1 1 5EF73240
 P 7600 3050
@@
 $EndComp
 $Comp
-L custom_power_rails:+7.5V #PWR?
+L vernier_current_driver:+7.5V #PWR?
 U 1 1 5EF92C6D
 P 7600 1650
@@
 $EndComp
 $Comp
-L custom_power_rails:+7.5V #PWR?
+L vernier_current_driver:+7.5V #PWR?
 U 1 1 5EFB1CFC
 P 950 6100
@@
 $EndComp
 $Comp
-L custom_power_rails:-7.5V #PWR?
+L vernier_current_driver:-7.5V #PWR?
 U 1 1 5EFF5F28
 P 950 7350
@@
 $EndComp
 $Comp
-L custom_power_rails:-7.5V #PWR?
+L vernier_current_driver:-7.5V #PWR?
 U 1 1 5F015856
 P 7600 5050
@@
 $EndComp
 $Comp
-L custom_power_rails:-7.5V #PWR?
+L vernier_current_driver:-7.5V #PWR?
 U 1 1 5F0250E3
 P 7600 3650
@@
 $EndComp
 $Comp
-L custom_power_rails:-7.5V #PWR?
+L vernier_current_driver:-7.5V #PWR?
 U 1 1 5F0349B1
 P 7600 2250

Commit message: Replace OPA2270 with OPA2210
These parts must have been missed somehow in 2617594b43217be702f357aa0c3cac4a60710900 and f9a9295af51ef93e9ca1b36aeebbcecdbb861685
Parts:
- U10: symbol Amplifier_Operational:OPA2277 -> vernier_current_driver:OPA2210
Changed lines of the file:
@@
 $EndComp
 $Comp
-L Amplifier_Operational:OPA2277 U10
+L vernier_current_driver:OPA2210 U10
 U 3 1 5EEB2ED9
 P 7700 3350
