File: Hardware/PCBs/Low_Current_Driver/MCU.sch (KiCad schematic (older format))
At the start: 13 parts, among them J9 Conn_01x02

Commit message: Switch to common shared library
Changed lines of the file:
@@
 Connection ~ 6050 2550
 $Comp
-L custom_power_rails:+12V_batt_post #PWR?
+L vernier_current_driver:+12V_batt_post #PWR?
 U 1 1 5EE2FEC9
 P 4700 2550
