File: Hardware/PCBs/Low_Current_Driver/Power.sch (KiCad schematic (older format))
At the start: 19 parts, among them U4 TPS7A470x, U5 TPS7A470x, U6 TPS7A33

Commit message: Switch to common shared library
Parts:
- U4, U5: symbol TPS74A4700:TPS7A470x -> vernier_current_driver:TPS7A470x
- U6: symbol TPS7A33:TPS7A33 -> vernier_current_driver:TPS7A33
Changed lines of the file:
@@
 	6650 5350 7050 5350
 $Comp
-L TPS7A33:TPS7A33 U6
+L vernier_current_driver:TPS7A33 U6
 U 1 1 5E321ECA
 P 5750 5250
@@
 	5250 5350 4350 5350
 $Comp
-L TPS74A4700:TPS7A470x U5
+L vernier_current_driver:TPS7A470x U5
 U 1 1 5E4EDE9C
 P 5750 3300
@@
 $EndComp
 $Comp
-L TPS74A4700:TPS7A470x U4
+L vernier_current_driver:TPS7A470x U4
 U 1 1 5E30DC9B
 P 5750 1200
@@
 	2950 1600 2800 1600
 $Comp
-L custom_power_rails:+7.5V #PWR?
+L vernier_current_driver:+7.5V #PWR?
 U 1 1 5EF1688E
 P 7300 800
@@
 $EndComp
 $Comp
-L custom_power_rails:-7.5V #PWR?
+L vernier_current_driver:-7.5V #PWR?
 U 1 1 5EF16888
 P 7400 5650
